File: PCB/HexiLux-v1.kicad_pcb (KiCad board)
At the start: 4 copper layers, 138.6 x 120 mm, 36 parts, among them U1 XIAO-ESP32-S3-DIP, U2 SN74AHCT1G125DBVR

Commit message: Start work on CAD
Parts:
- removed C3: WCAP-ATUL_6.3X11, WCAP-ATUL_6.3X11_DXL_100uF_35V:WCAP-ATUL_6.3X11_DXL_100uF_35V
- removed U3, U5, U6, U7, U8: ~, 3pin_female_header:3pin_female_header_out
- added C1: GRM31CD80J107MEA8L, 100uf_5V_1206:100uf_5V_1206, F.Cu at (100.3, 140.8)
- added G***: LOGO, Silkscreen:HexiLux-Logo, F.Cu at (115.3, 91.7)
- added G***: LOGO, Silkscreen:hackclub-logo, F.Cu at (104.4, 45.0)
- added G***: LOGO, Silkscreen:soup, B.Cu at (94.4, 124.5)
- added G***: LOGO, Silkscreen:hackclub-square, B.Cu at (117.1, 79.5)
- added J1: 10155435-00011LF, USBC-DigiKey-PD:AMPHENOL_10155435-00011LF, F.Cu at (136.5, 148.6)
- added R2: RC0603FR-075K1L, 5.1k_0603_DK:5.1k_0603_DK, F.Cu at (138.2, 141.2)
- added R4: RC0603FR-075K1L, 5.1k_0603_DK:5.1k_0603_DK, F.Cu at (135.2, 141.2)
- moved U2 28.0 mm to (102.0, 147.9)
Connections:
- S1 pad 2: (no net) -> BTN
- S1 pad 4: (no net) -> GND
Routing:
- net +3.3V: track 0.00 -> 66.4 mm
- net BTN: track 0.00 -> 59.2 mm
- net WS: track 0.00 -> 56.1 mm
- net SCK: track 0.00 -> 50.3 mm
- net SD: track 0.00 -> 42.5 mm
- net GND: track 0.00 -> 36.9 mm, vias 0 -> 20
- net Net-(D24-DOUT): track 0.00 -> 31.8 mm
- net Net-(D39-DOUT): track 0.00 -> 31.8 mm
- net Net-(D30-DOUT): track 0.00 -> 25.2 mm
- net Net-(D29-DOUT): track 0.00 -> 25.1 mm
- net Net-(D22-DOUT): track 0.00 -> 19.0 mm
- net Net-(D40-DOUT): track 0.00 -> 18.9 mm
- net Net-(D30-DIN): track 0.00 -> 18.9 mm
- net Net-(D25-DOUT): track 0.00 -> 18.9 mm
- net Net-(D35-DOUT): track 0.00 -> 18.9 mm
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- added copper zone on F.Cu, net +5V
- added copper zone on B.Cu, net GND
Other:
- copper layers 4 -> 2

Commit message: Update README
Connections:
- U1 pad 2: LIGHTSOUT -> unconnected-(U1-GPIO2/DA/A1-Pad2)_1
- U1 pad 4: unconnected-(U1-GPIO4/D3/A3-Pad4) -> LIGHTSOUT
Routing:
- net LIGHTSOUT: track 6.50 -> 11.9 mm
Changed lines of the file:
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@@
 	(net 33 "unconnected-(U1-GPIO5{slash}D4{slash}I2C_SDA-Pad5)")
 	(net 34 "unconnected-(U1-U0TXD{slash}D6{slash}TX-Pad7)")
-	(net 35 "unconnected-(U1-GPIO4{slash}D3{slash}A3-Pad4)")
+	(net 35 "unconnected-(U1-GPIO2{slash}DA{slash}A1-Pad2)")
 	(net 36 "unconnected-(U1-GPIO3{slash}D2{slash}A2-Pad3)_1")
 	(net 37 "unconnected-(U1-U0RXD{slash}D7{slash}RX-Pad8)_1")
@@
 	(net 44 "unconnected-(J1-SBU2-PadB8)")
 	(net 45 "Net-(J1-CC1)")
+	(net 46 "unconnected-(U1-GPIO3{slash}D2{slash}A2-Pad3)")
+	(net 47 "unconnected-(U1-GPIO5{slash}D4{slash}I2C_SDA-Pad5)_1")
+	(net 48 "unconnected-(U1-U0TXD{slash}D6{slash}TX-Pad7)_1")
+	(net 49 "unconnected-(U1-GPIO2{slash}DA{slash}A1-Pad2)_1")
+	(net 50 "unconnected-(U1-GPIO9{slash}D5{slash}I2C_SCL-Pad6)_1")
+	(net 51 "unconnected-(U1-U0RXD{slash}D7{slash}RX-Pad8)")
 	(footprint "5.1k_0603_DK:5.1k_0603_DK"
 		(layer "F.Cu")
@@
 			(layers "*.Cu" "*.Mask")
 			(remove_unused_layers no)
-			(net 31 "LIGHTSOUT")
+			(net 35 "unconnected-(U1-GPIO2{slash}DA{slash}A1-Pad2)")
 			(pinfunction "GPIO2/DA/A1")
-			(pintype "passive")
+			(pintype "passive+no_connect")
 		)
 		(pad "2" smd roundrect
@@
 			(layers "B.Cu" "B.Mask")
 			(roundrect_rratio 0.1)
-			(net 31 "LIGHTSOUT")
+			(net 49 "unconnected-(U1-GPIO2{slash}DA{slash}A1-Pad2)_1")
 			(pinfunction "GPIO2/DA/A1")
-			(pintype "passive")
+			(pintype "passive+no_connect")
 			(thermal_bridge_angle 45)
 		)
@@
 			(layers "B.Cu" "B.Mask")
 			(roundrect_rratio 0.1)
-			(net 36 "unconnected-(U1-GPIO3{slash}D2{slash}A2-Pad3)_1")
+			(net 46 "unconnected-(U1-GPIO3{slash}D2{slash}A2-Pad3)")
 			(pinfunction "GPIO3/D2/A2")
 			(pintype "passive+no_connect")
@@
 			(layers "*.Cu" "*.Mask")
 			(remove_unused_layers no)
-			(net 35 "unconnected-(U1-GPIO4{slash}D3{slash}A3-Pad4)")
+			(net 31 "LIGHTSOUT")
 			(pinfunction "GPIO4/D3/A3")
-			(pintype "passive+no_connect")
+			(pintype "passive")
 		)
 		(pad "4" smd roundrect
@@
 			(layers "B.Cu" "B.Mask")
 			(roundrect_rratio 0.1)
-			(net 35 "unconnected-(U1-GPIO4{slash}D3{slash}A3-Pad4)")
+			(net 31 "LIGHTSOUT")
 			(pinfunction "GPIO4/D3/A3")
-			(pintype "passive+no_connect")
+			(pintype "passive")
 			(thermal_bridge_angle 45)
 		)
@@
 			(layers "B.Cu" "B.Mask")
 			(roundrect_rratio 0.1)
-			(net 33 "unconnected-(U1-GPIO5{slash}D4{slash}I2C_SDA-Pad5)")
+			(net 47 "unconnected-(U1-GPIO5{slash}D4{slash}I2C_SDA-Pad5)_1")
 			(pinfunction "GPIO5/D4/I2C_SDA")
 			(pintype "passive+no_connect")
@@
 			(layers "B.Cu" "B.Mask")
 			(roundrect_rratio 0.1)
-			(net 32 "unconnected-(U1-GPIO9{slash}D5{slash}I2C_SCL-Pad6)")
+			(net 50 "unconnected-(U1-GPIO9{slash}D5{slash}I2C_SCL-Pad6)_1")
 			(pinfunction "GPIO9/D5/I2C_SCL")
 			(pintype "passive+no_connect")
@@
 			(layers "*.Cu" "*.Mask")
 			(remove_unused_layers no)
-			(net 34 "unconnected-(U1-U0TXD{slash}D6{slash}TX-Pad7)")
+			(net 48 "unconnected-(U1-U0TXD{slash}D6{slash}TX-Pad7)_1")
 			(pinfunction "U0TXD/D6/TX")
 			(pintype "passive+no_connect")
@@
 			(layers "*.Cu" "*.Mask")
 			(remove_unused_layers no)
-			(net 37 "unconnected-(U1-U0RXD{slash}D7{slash}RX-Pad8)_1")
+			(net 51 "unconnected-(U1-U0RXD{slash}D7{slash}RX-Pad8)")
 			(pinfunction "U0RXD/D7/RX")
 			(pintype "passive+no_connect")
@@
 	)
 	(segment
-		(start 103.933528 147.9)
-		(end 105.273529 146.559999)
+		(start 106.790529 139.154674)
+		(end 107.625529 139.154674)
+		(width 0.2)
+		(layer "B.Cu")
+		(net 31)
+	)
+	(segment
+		(start 103.255 147.9)
+		(end 103.548362 147.9)
 		(width 0.2)
 		(layer "B.Cu")
@@
 	)
 	(segment
-		(start 105.273529 145.509044)
-		(end 106.547899 144.234674)
+		(start 104.5 141.445203)
+		(end 106.790529 139.154674)
+		(width 0.2)
+		(layer "B.Cu")
+		(net 31)
+	)
+	(segment
+		(start 103.548362 147.9)
+		(end 104.5 146.948362)
 		(width 0.2)
 		(layer "B.Cu")
@@
 	)
 	(segment
-		(start 105.273529 146.559999)
-		(end 105.273529 145.509044)
+		(start 104.5 141.7)
+		(end 104.5 141.445203)
 		(width 0.2)
 		(layer "B.Cu")
@@
 	)
 	(segment
-		(start 106.547899 144.234674)
-		(end 107.625529 144.234674)
+		(start 104.5 146.948362)
+		(end 104.5 141.7)
 		(width 0.2)
 		(layer "B.Cu")
