File: PCB/HexiLux-v1.kicad_sch (KiCad schematic)
At the start: 36 parts, among them U1 XIAO-ESP32-S3-DIP, U2 SN74AHCT1G125DBVR

Commit message: Start work on CAD
Parts:
- removed C3: WCAP-ATUL_6.3X11, WCAP-ATUL_6.3X11_DXL_100uF_35V:WCAP-ATUL_6.3X11_DXL_100uF_35V, symbol WCAP-ATUL_6.3X11_100uF_35V:WCAP-ATUL_6.3X11
- removed U3, U5, U6, U7, U8: ~, 3pin_female_header:3pin_female_header_out, symbol 3pin_female_header:3pin_female_header_out
- added C1: GRM31CD80J107MEA8L, 100uf_5V_1206:100uf_5V_1206, symbol 100uf_5V_1206:GRM31CD80J107MEA8L
- added J1: 10155435-00011LF, USBC-DigiKey-PD:AMPHENOL_10155435-00011LF, symbol 10155435-00011LF:10155435-00011LF
- added R2, R4: RC0603FR-075K1L, 5.1k_0603_DK:5.1k_0603_DK, symbol 5.1k_0603_DK:RC0603FR-075K1L
Connections:
- net +5V: now also C1.1, J1.A4_B9 (VBUS), J1.B4_A9 (VBUS__1)
- net GND: now also C1.2, J1.A1_B12 (GND), J1.B1_A12 (GND__1), J1.SH1 (SHIELD), J1.SH2 (SHIELD__1), J1.SH3 (SHIELD__2), J1.SH4 (SHIELD__3), R2.2, R4.2
- new net: J1.A5 (CC1), R4.1
- new net: J1.B5 (CC2), R2.1
- no-connect marks 0 -> 12
Other:
- note added: "POWER"
- note removed: "HEADERS"

Commit message: Update README
Connections:
- net LIGHTSOUT: now also U1.4 (GPIO4/D3/A3); no longer U1.2 (GPIO2/DA/A1)
Changed lines of the file:
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@@
 	)
 	(no_connect
-		(at 41.91 64.77)
+		(at 41.91 57.15)
 	)
 	(no_connect
@@
 	(global_label "LIGHTSOUT"
 		(shape input)
-		(at 41.91 57.15 180)
+		(at 41.91 64.77 180)
 		(fields_autoplaced yes)
 		(effects
@@
 		)
 		(property "Intersheetrefs" "${INTERSHEET_REFS}"
-			(at 28.8857 57.15 0)
+			(at 28.8857 64.77 0)
 			(effects
 				(font
